File: Hardware/PORT0.kicad_sch (KiCad schematic)
At the start: 6 parts

Commit message: fixes for hierarchical sheets
Connections:
- net EN_3 is gone; now on net EN: R?.1
Changed lines of the file:
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@@
     (effects (font (size 1.27 1.27)) (justify left bottom))
   )
-  (label "EN_3" (at 82.55 66.04 0)
+  (label "EN" (at 82.55 66.04 0)
     (effects (font (size 1.27 1.27)) (justify left bottom))
   )
@@
     (pin "2")
   )
-  (symbol (lib_id "power:+5V") (at 110.49 41.91 0) (unit 1)
-    (in_bom yes) (on_board yes)
-    (property "Reference" "#PWR?" (id 0) (at 110.49 45.72 0)
+  (symbol (lib_id "power:+5V") (at 92.71 41.91 0) (unit 1)
+    (in_bom yes) (on_board yes) (fields_autoplaced)
+    (property "Reference" "#PWR?" (id 0) (at 92.71 45.72 0)
       (effects (font (size 1.27 1.27)) hide)
     )
-    (property "Value" "~" (id 1) (at 111.76 40.64 0)
-      (effects (font (size 1.27 1.27)) (justify left))
-    )
-    (property "Footprint" "" (id 2) (at 110.49 41.91 0)
+    (property "Value" "+5V" (id 1) (at 92.71 36.83 0))
+    (property "Footprint" "" (id 2) (at 92.71 41.91 0)
       (effects (font (size 1.27 1.27)) hide)
     )
-    (property "Datasheet" "" (id 3) (at 110.49 41.91 0)
+    (property "Datasheet" "" (id 3) (at 92.71 41.91 0)
       (effects (font (size 1.27 1.27)) hide)
     )
@@
     (pin "8")
   )
+  (symbol (lib_id "power:+5V") (at 110.49 41.91 0) (unit 1)
+    (in_bom yes) (on_board yes) (fields_autoplaced)
+    (property "Reference" "#PWR?" (id 0) (at 110.49 45.72 0)
+      (effects (font (size 1.27 1.27)) hide)
+    )
+    (property "Value" "+5V" (id 1) (at 110.49 36.83 0))
+    (property "Footprint" "" (id 2) (at 110.49 41.91 0)
+      (effects (font (size 1.27 1.27)) hide)
+    )
+    (property "Datasheet" "" (id 3) (at 110.49 41.91 0)
+      (effects (font (size 1.27 1.27)) hide)
+    )
+    (pin "1")
+  )
   (symbol (lib_id "Device:R_Small") (at 90.17 66.04 90) (unit 1)
     (in_bom yes) (on_board yes) (fields_autoplaced)
@@
     (pin "5")
   )
-  (symbol (lib_id "power:+5V") (at 92.71 41.91 0) (unit 1)
-    (in_bom yes) (on_board yes)
-    (property "Reference" "#PWR?" (id 0) (at 92.71 45.72 0)
-      (effects (font (size 1.27 1.27)) hide)
-    )
-    (property "Value" "~" (id 1) (at 86.36 40.64 0)
-      (effects (font (size 1.27 1.27)) (justify left))
-    )
-    (property "Footprint" "" (id 2) (at 92.71 41.91 0)
-      (effects (font (size 1.27 1.27)) hide)
-    )
-    (property "Datasheet" "" (id 3) (at 92.71 41.91 0)
-      (effects (font (size 1.27 1.27)) hide)
-    )
-    (pin "1")
-  )
 )
