File: Hardware/USB_C.kicad_sch (KiCad schematic)
At the start: 3 parts

Commit message: fixes for hierarchical sheets
Connections:
- net 5V renamed 5V_USB
Changed lines of the file:
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@@
     (stroke (width 0) (type default) (color 0 0 0 0))
   )
-  (hierarchical_label "GND" (shape input) (at 97.79 83.82 0)
+  (hierarchical_label "5V_USB" (shape input) (at 116.84 45.72 0)
     (effects (font (size 1.27 1.27)) (justify left))
   )
-  (hierarchical_label "5V" (shape input) (at 116.84 45.72 0)
-    (effects (font (size 1.27 1.27)) (justify left))
-  )
