File: Hardware/display.kicad_sch (KiCad schematic)
At the start: 0 parts

Commit message: included psu on pcb
Other:
- company: (none) -> ncAudio
Changed lines of the file:
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@@
 (kicad_sch (version 20211123) (generator eeschema)
   (paper "A4")
+  (title_block
+    (date "2022-12-27")
+    (rev "0.1")
+    (company "ncAudio")
+  )
 )
